Commit message: Fix create2 gazebo urdf

File: create_robot/create_description/urdf/create_2.urdf.xacro (robot description, xacro)
@@ -3,5 +3,5 @@
   xmlns:xacro="http://ros.org/wiki/xacro">
   <xacro:include filename="$(find create_description)/urdf/create_base.urdf.xacro" />
-  <xacro:include filename="$(find create_description)/urdf/create_2_gazebo.urdf.xacro" />
+  <xacro:include filename="$(find create_description)/urdf/create_base_gazebo.urdf.xacro" />
   <xacro:create_base wheel_separation="0.235" base_diameter="0.3485" version="2">
     <mesh filename="package://create_description/meshes/create_2.dae" />

File: create_robot/create_description/urdf/create_base_gazebo.urdf.xacro (robot description, xacro)
@@ -212,3 +212,35 @@
     </gazebo>
   </xacro:macro>
+  <gazebo reference="base_scan">
+    <material>Gazebo/FlatBlack</material>
+    <sensor type="ray" name="lds_lfcd_sensor">
+      <pose>0 0 0 0 0 0</pose>
+      <visualize>$(arg laser_visual)</visualize>
+      <update_rate>5</update_rate>
+      <ray>
+        <scan>
+          <horizontal>
+            <samples>360</samples>
+            <resolution>1</resolution>
+            <min_angle>0.0</min_angle>
+            <max_angle>6.28319</max_angle>
+          </horizontal>
+        </scan>
+        <range>
+          <min>0.120</min>
+          <max>3.5</max>
+          <resolution>0.015</resolution>
+        </range>
+        <noise>
+          <type>gaussian</type>
+          <mean>0.0</mean>
+          <stddev>0.01</stddev>
+        </noise>
+      </ray>
+      <plugin name="gazebo_ros_lds_lfcd_controller" filename="libgazebo_ros_laser.so">
+        <topicName>scan</topicName>
+        <frameName>base_scan</frameName>
+      </plugin>
+    </sensor>
+  </gazebo>
 </robot>
